File: USB-2-switch-and-hub.kicad_pcb (KiCad board)
At the start: 2 copper layers, 90 parts, among them J1 USB_C_Receptacle_USB2.0, J2 USB_A, J3 USB_A, J4 SWD, J7 USB_C_Receptacle_USB2.0, Q1 BSS138, Q2 BSS138, Q3 BSS138, SW1 SW_Push, SW3 SW_Push, U1 SRV05-4, U10 SRV05-4, U2 RP2040, U3 USB2514B_Bi, U4 SRV05-4, U5 SRV05-4, U6 W25Q128JVS, U8 TLV1117-33, Y1 24MHz, Y2 12MHz

Commit message: Assigned footprints
Parts:
- removed C11, C23, C24, C26, C27, C28, C30, C31: 100nF, Capacitor_SMD:C_0402_1005Metric_Pad0.74x0.62mm_HandSolder
- removed C25, C32, C33, C34: 10uF, Capacitor_SMD:C_1206_3216Metric_Pad1.33x1.80mm_HandSolder
- removed C29: 1uF, Capacitor_SMD:C_0603_1608Metric_Pad1.08x0.95mm_HandSolder
- removed Q1, Q2, Q3: BSS138, Package_TO_SOT_SMD:SOT-23
- removed R11, R20, R21, R22, R23: 10K, Resistor_SMD:R_0603_1608Metric_Pad0.98x0.95mm_HandSolder
- removed R13: 27, Capacitor_SMD:C_0402_1005Metric_Pad0.74x0.62mm_HandSolder
- removed R14, R15, R16: 1K, Resistor_SMD:R_0805_2012Metric_Pad1.20x1.40mm_HandSolder
- removed R17: DNI, Capacitor_SMD:C_0805_2012Metric_Pad1.18x1.45mm_HandSolder
- removed R18: 100, Resistor_SMD:R_0805_2012Metric_Pad1.20x1.40mm_HandSolder
- removed SW1, SW3: SW_Push, Button_Switch_THT:SW_PUSH_6mm_H5mm
- removed U1, U10: SRV05-4, Package_TO_SOT_SMD:SOT-23-6
- removed Y2: 12MHz, Crystal:Crystal_SMD_3225-4Pin_3.2x2.5mm_HandSoldering
- added C20: 10uF, Capacitor_SMD:C_1206_3216Metric_Pad1.33x1.80mm_HandSolder, F.Cu at (27.9, -14.6)
- added C21: 10uF, Capacitor_SMD:C_1206_3216Metric_Pad1.33x1.80mm_HandSolder, F.Cu at (27.9, -11.3)
- added C22: 10uF, Capacitor_SMD:C_1206_3216Metric_Pad1.33x1.80mm_HandSolder, F.Cu at (27.9, -7.91)
- added C5: 10uF, Capacitor_SMD:C_1206_3216Metric_Pad1.33x1.80mm_HandSolder, F.Cu at (27.9, -18.0)
- added C9: 100nF, Capacitor_SMD:C_0402_1005Metric_Pad0.74x0.62mm_HandSolder, F.Cu at (21.8, 11.1)
- added D2: D_Schottky, Diode_SMD:D_SOD-128, F.Cu at (-5.30, -8.00)
- added D5: D_Schottky, Diode_SMD:D_SOD-128, F.Cu at (-5.30, -3.95)
- added J3: USB_C_Receptacle_USB2.0, Connector_USB:USB_C_Receptacle_HRO_TYPE-C-31-M-12, F.Cu at (26.0, 0.91)
- added J5: USB_A, Connector_USB:USB_A_Molex_67643_Horizontal, F.Cu at (7.57, -34.8)
- added J6: USB_A, Connector_USB:USB_A_Molex_67643_Horizontal, F.Cu at (7.57, -17.5)
- added J7: USB_A, Connector_USB:USB_A_Molex_67643_Horizontal, F.Cu at (7.57, -0.22)
- added L2: 60R@100MHz, Inductor_SMD:L_1206_3216Metric, F.Cu at (28.2, -36.4)
- added L3: 60R@100MHz, Inductor_SMD:L_1206_3216Metric, F.Cu at (28.2, -33.0)
- added L4: 60R@100MHz, Inductor_SMD:L_1206_3216Metric, F.Cu at (28.2, -29.5)
- added L5: 60R@100MHz, Inductor_SMD:L_1206_3216Metric, F.Cu at (28.2, -26.1)
- added L6: 60R@100MHz, Inductor_SMD:L_1206_3216Metric, F.Cu at (28.2, -22.6)
- added R10: 12k, Resistor_SMD:R_0805_2012Metric_Pad1.20x1.40mm_HandSolder, F.Cu at (22.5, -6.36)
- added R3: 5.1k, Resistor_SMD:R_0805_2012Metric_Pad1.20x1.40mm_HandSolder, F.Cu at (22.5, -18.2)
- added R4: 5.1k, Resistor_SMD:R_0805_2012Metric_Pad1.20x1.40mm_HandSolder, F.Cu at (22.5, -15.2)
- added R8: 12k, Resistor_SMD:R_0805_2012Metric_Pad1.20x1.40mm_HandSolder, F.Cu at (22.5, -12.3)
- added R9: 12k, Resistor_SMD:R_0805_2012Metric_Pad1.20x1.40mm_HandSolder, F.Cu at (22.5, -9.31)
- added U2: USBLC6-2SC6, Package_TO_SOT_SMD:SOT-23-6, F.Cu at (22.7, -35.7)
- added U4: USBLC6-2SC6, Package_TO_SOT_SMD:SOT-23-6, F.Cu at (22.7, -31.1)
- added U5: USBLC6-2SC6, Package_TO_SOT_SMD:SOT-23-6, F.Cu at (22.7, -26.5)
- added U6: USBLC6-2SC6, Package_TO_SOT_SMD:SOT-23-6, F.Cu at (22.7, -21.9)
- added U7: TS3USB30EDGSR, Package_SO:VSSOP-10_3x3mm_P0.5mm, F.Cu at (23.9, 7.88)
- C21: value 1uF -> 10uF; footprint Capacitor_SMD:C_0603_1608Metric_Pad1.08x0.95mm_HandSolder -> Capacitor_SMD:C_1206_3216Metric_Pad1.33x1.80mm_HandSolder
- C22: value 100nF -> 10uF; footprint Capacitor_SMD:C_0402_1005Metric_Pad0.74x0.62mm_HandSolder -> Capacitor_SMD:C_1206_3216Metric_Pad1.33x1.80mm_HandSolder
- C5: value 22pF -> 10uF; footprint Capacitor_SMD:C_0402_1005Metric_Pad0.74x0.62mm_HandSolder -> Capacitor_SMD:C_1206_3216Metric_Pad1.33x1.80mm_HandSolder
- C9: value 22pF -> 100nF
- J3: value USB_A -> USB_C_Receptacle_USB2.0; footprint Connector_USB:USB_A_Molex_67643_Horizontal -> Connector_USB:USB_C_Receptacle_HRO_TYPE-C-31-M-12
- J4: value SWD -> Conn_01x03; footprint Connector_PinSocket_2.54mm:PinSocket_1x05_P2.54mm_Vertical -> Connector_PinHeader_2.54mm:PinHeader_1x03_P2.54mm_Vertical
- J7: value USB_C_Receptacle_USB2.0 -> USB_A; footprint Connector_USB:USB_C_Receptacle_HRO_TYPE-C-31-M-12 -> Connector_USB:USB_A_Molex_67643_Horizontal
- R10: value 100 -> 12k
- R3: value 27 -> 5.1k; footprint Capacitor_SMD:C_0402_1005Metric_Pad0.74x0.62mm_HandSolder -> Resistor_SMD:R_0805_2012Metric_Pad1.20x1.40mm_HandSolder
- R4: value 10K -> 5.1k; footprint Resistor_SMD:R_0603_1608Metric_Pad0.98x0.95mm_HandSolder -> Resistor_SMD:R_0805_2012Metric_Pad1.20x1.40mm_HandSolder
- R8, R9: value 56k -> 12k
- U2: value RP2040 -> USBLC6-2SC6; footprint Package_DFN_QFN:QFN-56-1EP_7x7mm_P0.4mm_EP3.2x3.2mm -> Package_TO_SOT_SMD:SOT-23-6
- U4, U5: value SRV05-4 -> USBLC6-2SC6
- U6: value W25Q128JVS -> USBLC6-2SC6; footprint Package_SO:SOIC-8_5.23x5.23mm_P1.27mm -> Package_TO_SOT_SMD:SOT-23-6
- moved J7 50.9 mm to (10.5, 25.1)
Connections:
- C21 pad 1: +1V1 -> +5V
- C22 pad 1: +3V3 -> +5V
- C5 pad 1: GND -> +3V3
- C5 pad 2: Net-(U2-XIN) -> GND
- C9 pad 1: GND -> +3V3
- C9 pad 2: Net-(C9-Pad2) -> GND
- J1 pad A4: VBUS -> Net-(D2-A)
- J1 pad A6: DUP+ -> DUP1+
- J1 pad A7: DUP- -> DUP1-
- J1 pad A9: VBUS -> Net-(D2-A)
- J1 pad B4: VBUS -> Net-(D2-A)
- J1 pad B6: DUP+ -> DUP1+
- J1 pad B7: DUP- -> DUP1-
- J1 pad B9: VBUS -> Net-(D2-A)
- J1 pad S1: GNDPWR -> Net-(J1-SHIELD)
- J2 pad 2: D1- -> Net-(J2-D-)
- J2 pad 3: D1+ -> Net-(J2-D+)
- J2 pad 4: GND -> Net-(J2-GND)
- J2 pad 5: GNDPWR -> GND
- J4 pad 1: RESET -> +3V3
- J4 pad 2: +3V3 -> SELECT
- L1 pad 2: GNDPWR -> Net-(J1-SHIELD)
- R10 pad 1: LED-POWER -> Net-(D7-A)
- R3 pad 1: D2+ -> Net-(J3-CC1)
- R3 pad 2: Net-(U2-USB_DP) -> GND
- R4 pad 1: TP4-CLK-3V3 -> Net-(J3-CC2)
- R4 pad 2: +3V3 -> GND
- R8 pad 1: Net-(J7-CC1) -> GND
- R8 pad 2: +5V -> SELECT
- R9 pad 1: Net-(J7-CC2) -> Net-(D6-A)
- R9 pad 2: +5V -> SELECT
- U2 pad 1: +3V3 -> Net-(J2-D+)
- U2 pad 2: SENSE5 -> GND
- U2 pad 3: SENSE0 -> Net-(J2-D-)
- U2 pad 4: SENSE3 -> D1-
- U2 pad 5: SENSE2 -> +5V
- U2 pad 6: SENSE4 -> D1+
- U4 pad 1: unconnected-(U4-IO1-Pad1) -> Net-(J5-D+)
- U4 pad 3: unconnected-(U4-IO2-Pad3) -> Net-(J5-D-)
- U4 pad 4: D3- -> D2-
- U4 pad 6: D3+ -> D2+
- U5 pad 1: unconnected-(U5-IO1-Pad1) -> Net-(J6-D+)
- U5 pad 3: unconnected-(U5-IO2-Pad3) -> Net-(J6-D-)
- U5 pad 4: D4- -> D3-
- U5 pad 6: D4+ -> D3+
- U6 pad 1: CS -> Net-(J7-D+)
- U6 pad 2: SD1 -> GND
- U6 pad 3: SD2 -> Net-(J7-D-)
- U6 pad 4: GND -> D4-
- U6 pad 5: SD0 -> +5V
- U6 pad 6: QSPI_CLK -> D4+

Commit message: Some work
Probably won't get prototyped anytime soon though
Parts:
- removed the J7 at (10.5, 25.1)
- added D6: LED, LED_THT:LED_D3.0mm_Clear, F.Cu at (-9.00, 12.0)
- added D7: LED, LED_THT:LED_D3.0mm_Clear, F.Cu at (-9.00, 17.5)
- moved J2 103.8 mm to (12.0, 40.0)
- moved H2 88.8 mm to (4.00, 46.0)
- moved J5 80.4 mm to (37.0, 40.0)
- moved J6 79.2 mm to (62.0, 40.0)
- moved C1 74.7 mm to (-49.5, -100.7)
- moved C12 74.7 mm to (-60.7, -77.3)
- moved C13 74.7 mm to (-60.7, -75.4)
- moved C14 74.7 mm to (-49.5, -94.0)
- moved C15 74.7 mm to (-49.5, -90.7)
- moved C17 74.7 mm to (-43.5, -100.7)
- moved C19 74.7 mm to (-43.5, -94.0)
- moved C20 74.7 mm to (-43.5, -90.7)
- moved C20 74.7 mm to (17.2, -88.5)
- moved C21 74.7 mm to (-32.9, -64.7)
- moved C22 74.7 mm to (17.2, -81.8)
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Other:
- board outline added: 100 x 50 mm
- copper layers 2 -> 4
- rule pad_to_mask_clearance: 0 -> 0.038
