File: USB-2-switch-and-hub.kicad_sch (KiCad schematic)
At the start: 74 parts, among them J1 USB_C_Receptacle_USB2.0, J2 USB_A, J3 USB_C_Receptacle_USB2.0, J4 Conn_01x03, J5 USB_A, J6 USB_A, J7 USB_A, U2 USBLC6-2SC6, U3 USB2514B_Bi, U4 USBLC6-2SC6, U5 USBLC6-2SC6, U6 USBLC6-2SC6, U7 TS3USB30EDGSR, U8 TLV1117-33, Y1 24MHz

Commit message: Assigned footprints
Parts:
- D2, D5: footprint (none) -> Diode_SMD:D_SOD-128
- J4: footprint (none) -> Connector_PinHeader_2.54mm:PinHeader_1x03_P2.54mm_Vertical
Changed lines of the file:
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@@
 			)
 		)
-		(property "Footprint" ""
+		(property "Footprint" "Diode_SMD:D_SOD-128"
 			(at 421.64 262.89 0)
 			(effects
@@
 			)
 		)
-		(property "Footprint" ""
+		(property "Footprint" "Diode_SMD:D_SOD-128"
 			(at 367.03 262.89 0)
 			(effects
@@
 			)
 		)
-		(property "Datasheet" " ~"
+		(property "Datasheet" "~"
 			(at 222.25 157.48 0)
 			(effects
@@
 			)
 		)
-		(property "Footprint" ""
+		(property "Footprint" "Connector_PinHeader_2.54mm:PinHeader_1x03_P2.54mm_Vertical"
 			(at 477.52 157.48 0)
 			(effects
@@
 			)
 		)
-		(property "Datasheet" " ~"
+		(property "Datasheet" "~"
 			(at 222.25 43.18 0)
 			(effects
@@
 			)
 		)
-		(property "Datasheet" " ~"
+		(property "Datasheet" "~"
 			(at 222.25 80.01 0)
 			(effects
@@
 			)
 		)
-		(property "Datasheet" " ~"
+		(property "Datasheet" "~"
 			(at 222.25 116.84 0)
 			(effects

Commit message: Some work
Probably won't get prototyped anytime soon though
Parts:
- removed C20, C21: 10uF, Capacitor_SMD:C_1206_3216Metric_Pad1.33x1.80mm_HandSolder, symbol Device:C
- removed D3, D4: RB060M-60TR, Diode_SMD:D_SOD-123, symbol Device:D_Schottky_Small
- removed J7: USB_A, Connector_USB:USB_A_Molex_67643_Horizontal, symbol Connector:USB_A
- removed L1, L2, L3, L4, L5, L6: 60R@100MHz, Inductor_SMD:L_1206_3216Metric, symbol Unified-Daughterboard-rescue:L_Core_Ferrite-Device
- added C11, C23, C24, C26, C27, C28, C44: 100nF, Capacitor_SMD:C_0805_2012Metric_Pad1.18x1.45mm_HandSolder, symbol Device:C
- added C29, C34, C35: 100nF, Capacitor_SMD:C_0402_1005Metric_Pad0.74x0.62mm_HandSolder, symbol Device:C_Small
- added C30, C31: 22pF, Capacitor_SMD:C_0402_1005Metric_Pad0.74x0.62mm_HandSolder, symbol Device:C
- added C32, C36: 10uF, Capacitor_SMD:C_1206_3216Metric_Pad1.33x1.80mm_HandSolder, symbol Device:C
- added C33, C37: 1uF, Capacitor_SMD:C_0603_1608Metric_Pad1.08x0.95mm_HandSolder, symbol Device:C
- added C38, C39, C40, C41, C42, C43: 100nF, Capacitor_SMD:C_0402_1005Metric_Pad0.74x0.62mm_HandSolder, symbol Device:C
- added D10, D11, D9: D_Schottky, Diode_SMD:D_SOD-128, symbol Device:D_Schottky
- added J3, J7: USB_C_Receptacle_USB2.0, Connector_USB:USB_C_Receptacle_HRO_TYPE-C-31-M-12, symbol Connector:USB_C_Receptacle_USB2.0
- added J8: SWD, Connector_PinSocket_2.54mm:PinSocket_1x05_P2.54mm_Vertical, symbol Connector_Generic:Conn_01x05
- added R11, R16: 56k, Resistor_SMD:R_0805_2012Metric_Pad1.20x1.40mm_HandSolder, symbol Device:R
- added R13, R14, R15, R17, R18, R20, R21: 330, Resistor_SMD:R_0805_2012Metric_Pad1.20x1.40mm_HandSolder, symbol Device:R
- added R22: DNI, Capacitor_SMD:C_0805_2012Metric_Pad1.18x1.45mm_HandSolder, symbol Device:R
- added R23, R27: 1K, Resistor_SMD:R_0805_2012Metric_Pad1.20x1.40mm_HandSolder, symbol Device:R_Small
- added R24, R25: 27, Capacitor_SMD:C_0402_1005Metric_Pad0.74x0.62mm_HandSolder, symbol Device:R
- added R26: 1K, Resistor_SMD:R_0805_2012Metric_Pad1.20x1.40mm_HandSolder, symbol Device:R
- added R28, R29: 5.1k, Resistor_SMD:R_0805_2012Metric_Pad1.20x1.40mm_HandSolder, symbol Device:R_Small
- added SW2, SW3: SW_Push, Button_Switch_THT:SW_PUSH_6mm_H5mm, symbol Switch:SW_Push
- added U1, U14: ~, symbol A-USB-2-switch-and-hub:OnSemi-NIS6452
- added U10: RP2040, Package_DFN_QFN:QFN-56-1EP_7x7mm_P0.4mm_EP3.2x3.2mm, symbol MCU_RaspberryPi:RP2040
- added U11, U12, U13: USBLC6-2SC6, Package_TO_SOT_SMD:SOT-23-6, symbol Power_Protection:USBLC6-2SC6
- added U9: W25Q128JVS, Package_SO:SOIC-8_5.23x5.23mm_P1.27mm, symbol Memory_Flash:W25Q128JVS
- added Y2: 12MHz, Crystal:Crystal_SMD_3225-4Pin_3.2x2.5mm_HandSoldering, symbol Device:Crystal_GND24
- D6, D7: footprint (none) -> LED_THT:LED_D3.0mm_Clear
- R8: value 12k -> 10k
- renumbered J3 to J2, J2 to J4, J4 to SW1
Connections:
- net +3V3: now also C29.1, C32.1, C36.1, C37.1, C38.1, C39.1, C40.1, C41.1, C42.1, C43.1, D10.2 (A), J8.2 (Pin_2), R22.2, R27.2, U10.1 (IOVDD), U10.10 (IOVDD), U10.22 (IOVDD), U10.33 (IOVDD), U10.42 (IOVDD), U10.43 (ADC_AVDD), U10.44 (VREG_IN), U10.48 (USB_VDD), U10.49 (IOVDD), U9.8 (VCC)
- net +5V: now also D10.1 (K), R11.2, R16.2, U11.5 (VBUS), U12.5 (VBUS), U13.5 (VBUS)
- net D4+: now also U6.4 (I/O2); no longer U6.6 (I/O1)
- net D4-: now also U6.6 (I/O1); no longer U6.4 (I/O2)
- net DUP1+: now also U13.4 (I/O2); no longer J1.A6 (D+), J1.B6 (D+)
- net DUP1-: now also U13.6 (I/O1); no longer J1.A7 (D-), J1.B7 (D-)
- net DUP2+: now also U12.4 (I/O2); no longer J2.A6 (D+), J2.B6 (D+)
- net DUP2-: now also U12.6 (I/O1); no longer J2.A7 (D-), J2.B7 (D-)
- net GND: now also J4.4 (GND), J5.4 (GND), J6.4 (GND), C11.2, C23.2, C24.2, C26.2, C27.2, C28.2, C29.2, C30.1, C31.1, C32.2, C33.2, C34.2, C35.2, C36.2, C37.2, C38.2, C39.2, C40.2, C41.2, C42.2, C43.2, C44.2, J3.A1 (GND), J3.A12 (GND), J3.B1 (GND), J3.B12 (GND), J7.A1 (GND), J7.A12 (GND), J7.B1 (GND), J7.B12 (GND), J8.3 (Pin_3), R13.2, R14.2, R15.2, R17.2, R18.2, R20.2, R21.2, R28.2, R29.1, SW2.1, SW3.1, U1.12 (GND), U1.13 (GND), U10.19 (TESTEN), U10.57 (GND), U11.2 (GND), U12.2 (GND), U13.2 (GND), U14.12 (GND), U14.13 (GND), U9.4 (GND), Y2.2, Y2.4; no longer J4.5 (Shield), J5.5 (Shield), J6.5 (Shield)
- net VBUS: now also D9.1 (K)
- net at J1.S1 (SHIELD): now also C26.1, R17.1
- net at U6.1 (I/O1): now also J7.A7 (D-), J7.B7 (D-)
- net at U6.3 (I/O2): now also J7.A6 (D+), J7.B6 (D+)
- net at J2.S1 (SHIELD): now also C27.1, R18.1
- new net: C31.2, R26.1, Y2.1
- new net: C24.1, J6.5 (Shield), R15.1
- new net: C28.1, J3.S1 (SHIELD), R20.1
- new net: J1.A6 (D+), J1.B6 (D+), U13.3 (I/O2)
- new net: J1.A7 (D-), J1.B7 (D-), U13.1 (I/O1)
- new net: R24.2, U10.47 (USB_DP)
- new net: C30.2, U10.20 (XIN), Y2.3
- new net: C23.1, J5.5 (Shield), R14.1
- new net: J2.A7 (D-), J2.B7 (D-), U12.1 (I/O1)
- new net: J2.A6 (D+), J2.B6 (D+), U12.3 (I/O2)
- new net: R25.2, U10.46 (USB_DM)
- new net: C11.1, J4.5 (Shield), R13.1
- new net: J3.A7 (D-), J3.B7 (D-), U11.1 (I/O1)
- new net: J3.A6 (D+), J3.B6 (D+), U11.3 (I/O2)
- new net: D9.2 (A), J3.A4 (VBUS), J3.A9 (VBUS), J3.B4 (VBUS), J3.B9 (VBUS)
- new net: R26.2, U10.21 (XOUT)
- new net: U14.1 (Vin), U14.2 (Vin), U14.3 (Vin)
- new net: U14.10 (Vout), U14.11 (Vout), U14.9 (Vout)
- new net: U1.1 (Vin), U1.2 (Vin), U1.3 (Vin)
- new net: U1.10 (Vout), U1.11 (Vout), U1.9 (Vout)
- new net: C44.1, J7.S1 (SHIELD), R21.1
- new net +1V1: C33.1, C34.1, C35.1, U10.23 (DVDD), U10.45 (VREG_VOUT), U10.50 (DVDD)
- new net CS: R22.1, R23.2, U10.56 (QSPI_SS), U9.1 (~{CS})
- new net DOWNSTREAM_CC1: J7.A5 (CC1), R11.1, U10.40 (GPIO28_ADC2)
- new net DOWNSTREAM_CC2: J7.B5 (CC2), R16.1, U10.41 (GPIO29_ADC3)
- new net DOWNSTREAM_CC_+5V: J7.A4 (VBUS), J7.A9 (VBUS), J7.B4 (VBUS), J7.B9 (VBUS)
- new net POWER_CC1: J3.A5 (CC1), R28.1, U10.38 (GPIO26_ADC0)
- new net POWER_CC2: J3.B5 (CC2), R29.2, U10.39 (GPIO27_ADC1)
- new net QSPI_CLK: U10.52 (QSPI_SCLK), U9.6 (CLK)
- new net RESET: J8.1 (Pin_1), R27.1, SW2.2, U10.26 (RUN)
- new net RP2040_D+: R24.1, U11.4 (I/O2)
- new net RP2040_D-: R25.1, U11.6 (I/O1)
- new net SD0: U10.53 (QSPI_SD0), U9.5 (DI(IO0))
- new net SD1: U10.55 (QSPI_SD1), U9.2 (DO(IO1))
- new net SD2: U10.54 (QSPI_SD2), U9.3 (IO2)
- new net SD3: U10.51 (QSPI_SD3), U9.7 (IO3)
- new net SWCLK: J8.5 (Pin_5), U10.24 (SWCLK)
- new net SWD: J8.4 (Pin_4), U10.25 (SWD)
- new net ~{USB_BOOT}: R23.1, SW3.2
- no-connect marks 15 -> 19
Other:
- note added: "Downstream USB ports"
- note added: "Power/RP2040 USB port"
- note added: "RESET"
- note added: "RP2040"
- note added: "Selector switch (connect to SPDT, with SELECT connected to the common pin)"
- note removed: "Downstream USB A ports"
- note removed: "Selector switch (connect to SPDT, with select connected to the common pin)"
- moved on the sheet: C18, C22, D1, D2, D5, F1, J1, J2, J4, J6, R1, R2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
